Commit message: ograniczenie ruchu obrotowego

File: simple_arm.urdf (robot description, URDF)
Before this commit: robot proste_ramie, 6 links, 5 joints
Joints:
- joint joint1: limit lower=-3.14 upper=3.14 effort=100 velocity=1 -> lower=-2.618 upper=2.618 effort=100 velocity=1

Commit message: Refactor URDF for robotic arm with updated properties
Updated materials, dimensions, and properties for the robotic arm's URDF file. Adjusted mass, inertia, and added visual elements for gripper and joints.

File: simple_arm.urdf (robot description, URDF)
Before this commit: robot proste_ramie, 6 links, 5 joints
Links:
- link base_link: mass 10 -> 80; geometry collision cylinder length=0.16 radius=0.36; visual cylinder length=0.06 radius=0.24
- link gripper_link: mass None -> 1.2; geometry collision box size=0.2 0.044 0.14; visual box size=0.02 0.028 0.02
- link link1: mass 2 -> 16; geometry collision cylinder length=0.76 radius=0.09; visual cylinder length=0.08 radius=0.11
- link link2: mass 1.5 -> 9.6; geometry collision cylinder length=0.52 radius=0.072; visual cylinder length=0.06 radius=0.092
- link link3: mass 0.5 -> 4.8; geometry collision cylinder length=0.32 radius=0.056; visual cylinder length=0.32 radius=0.056
- link wrist_link: mass None -> 2; geometry collision cylinder length=0.14 radius=0.044; visual box size=0.2 0.12 0.036
Joints:
- joint joint1: axis 0 0 1 -> 0 0 2; limit lower=-2.618 upper=2.618 effort=100 velocity=1 -> lower=-2.618 upper=2.618 effort=300 velocity=1.2; origin xyz=0 0 0.05 rpy=0 0 0 -> xyz=0 0 0.14 rpy=0 0 0
- joint joint2: axis 0 1 0 -> 0 2 0; limit lower=-1.57 upper=1.57 effort=100 velocity=1 -> lower=-1.57 upper=1.57 effort=240 velocity=1.2; origin xyz=0 0 0.4 rpy=0 0 0 -> xyz=0 0 0.78 rpy=0 0 0
- joint joint3: axis 0 1 0 -> 0 2 0; limit lower=-1.57 upper=1.57 effort=100 velocity=1 -> lower=-1.57 upper=1.57 effort=160 velocity=1.5; origin xyz=0 0 0.3 rpy=0 0 0 -> xyz=0 0 0.54 rpy=0 0 0
- joint joint_gripper_fix: origin xyz=0 0 0.1 rpy=0 0 0 -> xyz=0 0 0.18 rpy=0 0 0
- joint joint_wrist: axis 0 1 0 -> 0 2 0; limit lower=-1.57 upper=1.57 effort=100 velocity=1 -> lower=-1.57 upper=1.57 effort=100 velocity=2.0; origin xyz=0 0 0.2 rpy=0 0 0 -> xyz=0 0 0.34 rpy=0 0 0

Commit message: Pozwól ramieniu dosięgnąć ziemi bez zmian wizualnych
Obniżono punkt obrotu joint2 o 0.30 m i wydłużono segment joint2->joint3
o 0.30 m, kompensując przesunięcie wizualizacji link2, dzięki czemu poza
spoczynkowa wygląda identycznie. Końcówka chwytaka sięga teraz poziomu
podłoża (fingertip z = -0.04 m zamiast 0.26 m). Obniżono też dolny limit
suwaka 'Ramię Cel Z' z 0.1 do 0.0, aby ziemia była osiągalna przez IK.

Co-authored-by: Bartosz Topa <Boros240@users.noreply.github.com>

File: simple_arm.urdf (robot description, URDF)
Before this commit: robot proste_ramie, 6 links, 5 joints
Joints:
- joint joint2: origin xyz=0 0 0.78 rpy=0 0 0 -> xyz=0 0 0.48 rpy=0 0 0
- joint joint3: origin xyz=0 0 0.54 rpy=0 0 0 -> xyz=0 0 0.84 rpy=0 0 0

Commit message: Adjust dimensions and positions in simple_arm.urdf

File: simple_arm.urdf (robot description, URDF)
Before this commit: robot proste_ramie, 6 links, 5 joints
Links:
- link link1: geometry collision cylinder length=0.38 radius=0.09; visual cylinder length=0.08 radius=0.11
Joints:
- joint joint2: origin xyz=0 0 0.78 rpy=0 0 0 -> xyz=0 0 0.39 rpy=0 0 0
