Commit message: komit

File: cube.urdf (robot description, URDF)
Before this commit: robot cube, 1 links, 0 joints
Links:
- link cube_link: mass 1.0 -> 0.05

Commit message: fix: dzialajacy Pick&Place A->B (poprawny IK, zbieznosc ruchu, zasieg)
Problem: ramie nie dochodzilo do punktu A i nie podnosilo kostki.
Przyczyny i poprawki (zweryfikowane testem headless w PyBullet DIRECT):

- move_ee_to: IK wywolywany bez limitow stawow zwracal katy poza zakresem,
  a ruch konczyl sie po stalej liczbie krokow mimo niedojechania; current_angles
  ustawiano na wartosci 'zyczeniowe' -> kumulacja bledu. Teraz IK dostaje
  lowerLimits/upperLimits/jointRanges/restPoses, a petla czeka az realne katy
  stawow osiagna cel i zapisuje rzeczywisty odczyt.
- cube.urdf: kostka zmniejszona 0.3 -> 0.16 m (chwytak nie odpychal jej bokiem).
- PickAndPlaceController: podejscie z gory + prawidlowa wysokosc chwytu/odlozenia.
- GRAB_THRESHOLD podniesiony (koncowka zawisa kilka cm nad kostka).
- Domyslne punkty A/B i spawn kostki w realnym zasiegu ramienia (promien ~0.45).
- RobotSimulation(gui=False) + zabezpieczenie audio -> testowalnosc headless.

Test integracyjny: kostka przenoszona z A do B z bledem <=12 mm dla ruchow
w sektorze przednim/bocznym.

Co-authored-by: Bartosz Topa <Boros240@users.noreply.github.com>

File: cube.urdf (robot description, URDF)
Before this commit: robot cube, 1 links, 0 joints
Links:
- link cube_link: mass 0.05 -> 0.2; geometry collision box size=0.16 0.16 0.16; visual box size=0.16 0.16 0.16

Commit message: fix: niezawodne chwytanie i odkladanie w Pick&Place (TCP, chwytak, kolizje)
Problemy zgloszone: robot nie opuszczal kostki na koncu, zle podchodzil i nie
lapal w punkcie A, a chwycona kostka lewitowala obok chwytaka.

Naprawy (zweryfikowane symulacja PyBullet headless, 5 tras A->B):
- simple_arm.urdf: SKROCONO element pionowy link1 (0.76 -> 0.44), dzieki czemu
  'bark' jest nizej i ramie REALNIE siega kostki lezacej na podlodze.
- simple_arm.urdf: WIEKSZY chwytak - dwa szersze/dluzsze palce rozstawione na
  +-0.10 m z PRZERWA w srodku oraz OSOBNE bryly kolizji per palec (kostka
  wchodzi miedzy palce, nie jest odpychana plaska bryla).
- Dodano wirtualny punkt narzedziowy TCP miedzy palcami; IK i dystans chwytania
  liczone wzgledem TCP -> chwytak trafia dokladnie w srodek kostki (offset ~5mm,
  koniec lewitacji). Prog chwytania zmniejszony 0.4 -> 0.1.
- Na czas sekwencji wylaczane sa kolizje robot<->kostka oraz palce<->podloga
  (palce moga zejsc do kostki na podlodze, bez odpychania).
- Naprawiono OPUSZCZANIE: wiez usuwany, a kolizje przywracane DOPIERO po
  odsunieciu ramienia w gore (palce nie odbijaja kostki przy puszczeniu).
- Kostka 0.16 -> 0.12 m (wygodnie miedzy palce); spawn/A/B i prześwit zaktualizowane.

Co-authored-by: Bartosz Topa <Boros240@users.noreply.github.com>

File: cube.urdf (robot description, URDF)
Before this commit: robot cube, 1 links, 0 joints
Links:
- link cube_link: geometry collision box size=0.12 0.12 0.12; visual box size=0.12 0.12 0.12

File: simple_arm.urdf (robot description, URDF)
Before this commit: robot proste_ramie, 6 links, 5 joints
Links:
- added link tcp_link, mass 0.001
- link gripper_link: geometry collision box size=0.04 0.05 0.16; collision box size=0.04 0.05 0.16
- link link1: geometry collision cylinder length=0.44 radius=0.09; visual cylinder length=0.08 radius=0.11
Joints:
- added joint joint_tcp: type fixed, parent gripper_link, child tcp_link, origin xyz=0 0 0.10 rpy=0 0 0
- joint joint2: origin xyz=0 0 0.78 rpy=0 0 0 -> xyz=0 0 0.46 rpy=0 0 0
